Commit message: fixed urdf for r2

File: exp_r2_sim/urdf/r2.ign.xacro (robot description, xacro)
@@ -19,5 +19,5 @@
         <wheel_separation>0.5735</wheel_separation>
         <wheel_radius>0.31</wheel_radius>
-        <topic>/cmd_vel</topic>
+        <topic>r2/cmd_vel</topic>
         <min_velocity>-1</min_velocity>
         <max_velocity>1</max_velocity>
@@ -25,5 +25,5 @@
         <max_acceleration>1.16</max_acceleration>
         <odom_topic>/odom</odom_topic>
-        <child_frame_id>${robot_namespace}/base_footprint</child_frame_id>
+        <child_frame_id>${robot_namespace}/base_link</child_frame_id>
       </plugin>
       <!-- Publish robot state information -->
@@ -91,7 +91,7 @@
                 filename="ignition-gazebo-joint-state-publisher-system"
                 name="ignition::gazebo::systems::JointStatePublisher">
-                <topic>joint_states</topic>
+                <topic>r2/joint_states</topic>
         </plugin>
-    </gazebo>
+        </gazebo>
         <gazebo reference='${robot_namespace}/imu_sensor'>
             <sensor name=

File: exp_r2_sim/urdf/r2.xacro (robot description, xacro)
@@ -1,4 +1,5 @@
 <?xml version='1.0' encoding='utf-8'?>
 <robot name="r2" xmlns:xacro="http://ros.org/wiki/xacro">
+    <pose>0 0 1.5 0 0 0</pose>
     <xacro:macro name="r2" params="robot_namespace">
         <xacro:property name="r2_prefix_stl" value="file://$(find exp_r2_sim)/meshes"/>
@@ -90,6 +91,6 @@
             </visual>
         </link>
-        <joint name='${robot_namespace}/Center Pivot' type='fixed'>
-            <origin xyz='-0.047625 0 -0.0254' rpy='1.5708 -0 0'/>
+        <joint name='${robot_namespace}/Center Pivot' type='revolute'>
+            <origin xyz='-0.047625 0 -0.0254' rpy='0 -0 0'/>
             <parent link='${robot_namespace}/base_link'/>
             <child link='${robot_namespace}/Rear_Rocker_Link'/>

Commit message: .

File: exp_r2_sim/urdf/r2.ign.xacro (robot description, xacro)
@@ -25,4 +25,5 @@
         <max_acceleration>1.16</max_acceleration>
         <odom_topic>/odom</odom_topic>
+        <odometry_frame>odom</odometry_frame>
         <child_frame_id>${robot_namespace}/base_link</child_frame_id>
       </plugin>

File: exp_r2_sim/urdf/r2.xacro (robot description, xacro)
@@ -26,8 +26,30 @@
             </collision>
             <visual name='base_link_visual'>
-                <origin xyz='0 0 0' rpy='0 0 -1.5708'/>
-                <geometry>
-                    <mesh filename='${r2_prefix_stl}/cube.STL' scale='1 1 1'/>
-                </geometry>
+                <origin xyz='0.180 0 0.24' rpy='0 0 -1.5708'/>
+                <geometry>
+                    <mesh filename='${r2_prefix_stl}/r2.dae'>
+                        <submesh>
+                            <name>BodyFront</name>
+                            <center>true</center>
+                        </submesh>
+                    </mesh>
+                </geometry>
+            <material>
+              <diffuse>1.0 1.0 1.0</diffuse>
+              <specular>1.0 1.0 1.0</specular>
+              <pbr>
+                  <metal>
+                    <albedo_map>file://$(find exp_r2_sim)/models/materials/textures/R2_Albedo.png</albedo_map>
+                      <metalness_map>file://$(find exp_r2_sim)/models/materials/textures/R2_Metalness.png</metalness_map>
+                      <roughness_map>file://$(find exp_r2_sim)/models/materials/textures/R2_Roughness.png</roughness_map>
+                  </metal>
+              </pbr>
+              <!-- fallback to script if no PBR support-->
+              <script>
+                  <uri>file://$(find exp_r2_sim)/models/materials/scripts/</uri>
+                  <uri>file://$(find exp_r2_sim)/models/materials/textures/</uri>
+                  <name>UrbanTile/R2_Diffuse</name>
+              </script>
+          </material>
             </visual>
             <visual name='base_link_fixed_joint_lump__sensor_payload_link_visual_1'>
